Commit message: Day 8 - adding a tray to krytn
- in `src/bar_examples/krytn/robot_description/krytn.urdf.xacro`
- new package `src/krytn_tray/` generated with FreeCAD CROSS

krytn_tray/
├── CMakeLists.txt
├── launch
│   ├── description.launch.py
│   ├── display.launch.py
│   └── gazebo.launch.py
├── meshes
│   ├── krytn_tray_ex_Body.dae
│   ├── krytn_tray_ex_caster_wheel.dae.dae
│   ├── krytn_tray_ex_collision_base_footprint_.dae
│   ├── krytn_tray_ex_front_wheel.dae.dae
│   ├── krytn_tray_ex_lidar_2d_v1.dae.dae
│   ├── krytn_tray_ex_magni_body.dae.dae
│   ├── krytn_tray_ex_realsense.dae.dae
│   └── krytn_tray_ex_visual_base_footprint_.dae
├── package.xml
├── rviz
│   └── robot_description.rviz
└── urdf
    └── krytn.urdf

File: src/bar_examples/krytn/robot_description/krytn.urdf.xacro (robot description, xacro)
@@ -11,4 +11,30 @@
     <origin xyz="0 0 0.15" rpy="0 0 0" />
   </xacro:lidar_2d>
+<!-- krytn_tray link-->
+  <link name="krytn_tray">
+    <visual>
+      <!--Krytn_tray_part/Body.-->
+      <origin rpy="0.0 -0.0 0.0" xyz="0.0 0.0 0.0"/>
+      <geometry>
+        <mesh filename="package://krytn_tray/meshes/krytn_tray_ex_Body.dae"/>
+      </geometry>
+    </visual>
+    <collision>
+      <!--Krytn_tray_part/Body.-->
+      <origin rpy="0.0 -0.0 0.0" xyz="0.0 0.0 0.0"/>
+      <geometry>
+        <mesh filename="package://krytn_tray/meshes/krytn_tray_ex_Body.dae"/>
+      </geometry>
+    </collision>
+    <xacro:box_inertial_with_origin x="0.400" y="0.280" z="0.220" mass="1.0">
+      <origin xyz="0.0 0.0 0.0" rpy="0 0 0" />
+    </xacro:box_inertial_with_origin>
+  </link>
+  <!-- tray_joint-->
+ <joint name="krytn_joint" type="fixed">
+    <parent link="base_link"/>
+    <child link="krytn_tray"/>
+    <origin rpy="0.0 -0.0 0.0" xyz="0.052 0.0 0.264"/>
+  </joint>
   <!-- Configure Control of Joints -->
   <ros2_control name="Krytn" type="system">
