Commit message: Troubleshooting: Changes from John's PR in Niacriza repo and other
in src/my_robot_arm/
 - new urdf/my_robot_arm.urdf_bkp.xacro - backup of my version
 - new launch/gazebo.launch_bkp.py - backup of my version
 - in ​urdf/my_robot_arm.urdf.xacro - pull request
​ - in launch/gazebo.launch.py - pull request
See: https://github.com/Niacriza/my_robot_arm/pulls

in src/my_robot_arm_moveit/
 - in package.xml - uncomment gazebo dependencies

File: src/my_robot_arm/urdf/my_robot_arm.urdf_bkp.xacro (robot description, xacro)
@@ -67,8 +67,10 @@
       <plugin>gz_ros2_control/GazeboSimSystem</plugin>
     </hardware>
+    <xacro:property name="initial_positions_file" value="$(find my_robot_arm_moveit)/config/initial_positions.yaml" />
+    <xacro:property name="initial_positions" value="${xacro.load_yaml(initial_positions_file)['initial_positions']}"/>
     <joint name="ur5_shoulder_pan_joint">
         <command_interface name="position"/>
         <state_interface name="position">
-          <param name="initial_value">0.0</param>
+          <param name="initial_value">${initial_positions['ur5_shoulder_pan_joint']}</param>
         </state_interface>
         <state_interface name="velocity"/>
@@ -77,5 +79,5 @@
         <command_interface name="position"/>
         <state_interface name="position">
-          <param name="initial_value">0.0</param>
+          <param name="initial_value">${initial_positions['ur5_shoulder_lift_joint']}</param>
         </state_interface>
         <state_interface name="velocity"/>
@@ -84,5 +86,5 @@
         <command_interface name="position"/>
         <state_interface name="position">
-          <param name="initial_value">0.0</param>
+          <param name="initial_value">${initial_positions['ur5_elbow_joint']}</param>
         </state_interface>
         <state_interface name="velocity"/>
@@ -91,5 +93,5 @@
         <command_interface name="position"/>
         <state_interface name="position">
-          <param name="initial_value">0.0</param>
+          <param name="initial_value">${initial_positions['ur5_wrist_1_joint']}</param>
         </state_interface>
         <state_interface name="velocity"/>
@@ -98,5 +100,5 @@
         <command_interface name="position"/>
         <state_interface name="position">
-          <param name="initial_value">0.0</param>
+          <param name="initial_value">${initial_positions['ur5_wrist_2_joint']}</param>
         </state_interface>
         <state_interface name="velocity"/>
@@ -105,5 +107,5 @@
         <command_interface name="position"/>
         <state_interface name="position">
-          <param name="initial_value">0.0</param>
+          <param name="initial_value">${initial_positions['ur5_wrist_3_joint']}</param>
         </state_interface>
         <state_interface name="velocity"/>
@@ -112,5 +114,5 @@
         <command_interface name="position"/>
         <state_interface name="position">
-          <param name="initial_value">0.0</param>
+          <param name="initial_value">${initial_positions['finger_joint']}</param>
         </state_interface>
         <state_interface name="velocity"/>
