Commit message: Day 15 configure arm with MoveIt
in src/my_robot_arm:
​ - in config/ros2_control.yaml - configure arm_controller

​ - in launch/gazebo.launch.py -
     launch arm_controller,
     launch move_group and rviz with moveit,
     set use_rviz default to false

​ - in urdf/my_robot_arm.urdf.xacro - add arm joints and
     xacro properties to read initial_positions.yaml
​
in src/my_robot_arm_moveit:

 - in config/initial_positions.yaml - replace every 0 with 0.0 just in case

​ - in config/joint_limits.yaml - set acceleration limits for all joints,
     and increase max_velocity to 1000.0 for finger_joint

 - in launch/move_group.launch.py - add capabilities bug fix

File: src/my_robot_arm/urdf/my_robot_arm.urdf.xacro (robot description, xacro)
@@ -67,10 +67,54 @@
       <plugin>gz_ros2_control/GazeboSimSystem</plugin>
     </hardware>
+    <xacro:property name="initial_positions_file" value="$(find my_robot_arm_moveit)/config/initial_positions.yaml" />
+    <xacro:property name="initial_positions" value="${xacro.load_yaml(initial_positions_file)['initial_positions']}"/>
+    <joint name="ur5_shoulder_pan_joint">
+        <command_interface name="position"/>
+        <state_interface name="position">
+          <param name="initial_value">${initial_positions['ur5_shoulder_pan_joint']}</param>
+        </state_interface>
+        <state_interface name="velocity"/>
+    </joint>
+    <joint name="ur5_shoulder_lift_joint">
+        <command_interface name="position"/>
+        <state_interface name="position">
+          <param name="initial_value">${initial_positions['ur5_shoulder_lift_joint']}</param>
+        </state_interface>
+        <state_interface name="velocity"/>
+    </joint>
+    <joint name="ur5_elbow_joint">
+        <command_interface name="position"/>
+        <state_interface name="position">
+          <param name="initial_value">${initial_positions['ur5_elbow_joint']}</param>
+        </state_interface>
+        <state_interface name="velocity"/>
+    </joint>
+    <joint name="ur5_wrist_1_joint">
+        <command_interface name="position"/>
+        <state_interface name="position">
+          <param name="initial_value">${initial_positions['ur5_wrist_1_joint']}</param>
+        </state_interface>
+        <state_interface name="velocity"/>
+    </joint>
+    <joint name="ur5_wrist_2_joint">
+        <command_interface name="position"/>
+        <state_interface name="position">
+          <param name="initial_value">${initial_positions['ur5_wrist_2_joint']}</param>
+        </state_interface>
+        <state_interface name="velocity"/>
+    </joint>
+    <joint name="ur5_wrist_3_joint">
+        <command_interface name="position"/>
+        <state_interface name="position">
+          <param name="initial_value">${initial_positions['ur5_wrist_3_joint']}</param>
+        </state_interface>
+        <state_interface name="velocity"/>
+    </joint>
     <joint name="finger_joint">
-      <command_interface name="position"/>
-      <state_interface name="position">
-        <param name="initial_value">0.0</param>
-      </state_interface>
-      <state_interface name="velocity"/>
+        <command_interface name="position"/>
+        <state_interface name="position">
+          <param name="initial_value">${initial_positions['finger_joint']}</param>
+        </state_interface>
+        <state_interface name="velocity"/>
     </joint>
   </ros2_control>

Commit message: Day 17 - add realsense camera (Not working)
In `src/my_robot_arm/urdf/my_robot_arm.urdf.xacro`:
 * add the xacro include and macro for the realsense camera

In `src/my_robot_arm/launch/gazebo.launch.py`:
 * add a `name` argument to the `robot` Node
 * add realsense stuff to the bridge
 * add a static publisher

No error messages but the PointCloud is not showing
Pushed to show to the instructor

File: src/my_robot_arm/urdf/my_robot_arm.urdf.xacro (robot description, xacro)
@@ -1,29 +1,39 @@
 <?xml version='1.0' encoding='utf-8'?>
 <robot xmlns:xacro="http://www.ros.org/wiki/xacro" name="my_robot_arm">
-    <xacro:include filename="$(find magni_description)/urdf/inertial.xacro" />
-    <!-- Include a UR05 -->
-    <xacro:include filename="$(find ur_description)/urdf/ur_macro.xacro" />
-    <xacro:arg name="ur_type" default="ur5e"/>
-    <xacro:ur_robot name="ur5" tf_prefix="ur5_" parent="world" joint_limits_parameters_file="$(find ur_description)/config/$(arg ur_type)/joint_limits.yaml" kinematics_parameters_file="$(find ur_description)/config/$(arg ur_type)/default_kinematics.yaml" physical_parameters_file="$(find ur_description)/config/$(arg ur_type)/physical_parameters.yaml" visual_parameters_file="$(find ur_description)/config/$(arg ur_type)/visual_parameters.yaml">
-        <origin xyz="-0.1 0 0.15" rpy="${pi} 0 0" />
-    </xacro:ur_robot>
-    <link name="world" />
-  <!--Generated by CROSS, a ROS Workbench for FreeCAD (https://github.com/galou/freecad.cross)-->
+  <xacro:include filename="$(find magni_description)/urdf/inertial.xacro" />
+  <xacro:include filename="$(find sensors)/realsense_d435/realsense.urdf.xacro" />
+  <xacro:realsense world_link_name="world">
+    <origin xyz="0 1.0 1.2" rpy="0 ${pi/4} -${pi/2}" />
+  </xacro:realsense>
+  <!-- Include a UR05 -->
+  <xacro:include filename="$(find ur_description)/urdf/ur_macro.xacro" />
+  <xacro:arg name="ur_type" default="ur5e" />
+  <xacro:ur_robot name="ur5" tf_prefix="ur5_" parent="world"
+    joint_limits_parameters_file="$(find ur_description)/config/$(arg ur_type)/joint_limits.yaml"
+    kinematics_parameters_file="$(find ur_description)/config/$(arg ur_type)/default_kinematics.yaml"
+    physical_parameters_file="$(find ur_description)/config/$(arg ur_type)/physical_parameters.yaml"
+    visual_parameters_file="$(find ur_description)/config/$(arg ur_type)/visual_parameters.yaml">
+    <origin xyz="-0.1 0 0.15" rpy="${pi} 0 0" />
+  </xacro:ur_robot>
+  <link name="world" />
+  <!--Generated
+  by CROSS, a ROS Workbench for FreeCAD (https://github.com/galou/freecad.cross)-->
   <link name="base_link">
     <visual>
       <!--base_link_part/Body.-->
-      <origin rpy="0.0 -0.0 0.0" xyz="0.0 0.0 0.0"/>
+      <origin rpy="0.0 -0.0 0.0" xyz="0.0 0.0 0.0" />
       <geometry>
-        <mesh filename="package://my_robot_arm/meshes/gripper_base_link_body.dae"/>
+        <mesh filename="package://my_robot_arm/meshes/gripper_base_link_body.dae" />
       </geometry>
     </visual>
     <collision>
       <!--base_link_part/Body.-->
-      <origin rpy="0.0 -0.0 0.0" xyz="0.0 0.0 0.0"/>
+      <origin rpy="0.0 -0.0 0.0" xyz="0.0 0.0 0.0" />
       <geometry>
-        <mesh filename="package://my_robot_arm/meshes/gripper_base_link_body.dae"/>
+        <mesh filename="package://my_robot_arm/meshes/gripper_base_link_body.dae" />
       </geometry>
     </collision>
-    <!--cylinder 50mm radius 150mm height 1.0kg, offset by -50mm in y, rotated 90deg in roll-->
+    <!--cylinder
+    50mm radius 150mm height 1.0kg, offset by -50mm in y, rotated 90deg in roll-->
     <xacro:cylinder_inertial_with_origin radius="0.05" length="0.15" mass="1.0">
       <origin xyz="0 -0.05 0" rpy="${pi/2} 0 0" />
@@ -33,17 +43,18 @@
     <visual>
       <!--finger_part/Body001.-->
-      <origin rpy="0.0 -0.0 0.0" xyz="0.0 0.0 0.0"/>
+      <origin rpy="0.0 -0.0 0.0" xyz="0.0 0.0 0.0" />
       <geometry>
-        <mesh filename="package://my_robot_arm/meshes/gripper_finger_body.dae"/>
+        <mesh filename="package://my_robot_arm/meshes/gripper_finger_body.dae" />
       </geometry>
     </visual>
     <collision>
       <!--finger_part/Body001.-->
-      <origin rpy="0.0 -0.0 0.0" xyz="0.0 0.0 0.0"/>
+      <origin rpy="0.0 -0.0 0.0" xyz="0.0 0.0 0.0" />
       <geometry>
-        <mesh filename="package://my_robot_arm/meshes/gripper_finger_body.dae"/>
+        <mesh filename="package://my_robot_arm/meshes/gripper_finger_body.dae" />
       </geometry>
     </collision>
-    <!--box 40x30x90mm 0.1kg, offset by -40mm in x, rotated 90deg in roll -->
+    <!--box
+    40x30x90mm 0.1kg, offset by -40mm in x, rotated 90deg in roll -->
     <xacro:box_inertial_with_origin x="0.04" y="0.03" z="0.09" mass="0.1">
       <origin xyz="-0.04 0.0 0.0" rpy="${pi/2} 0 0" />
@@ -51,9 +62,9 @@
   </link>
   <joint name="finger_joint" type="prismatic">
-    <parent link="base_link"/>
-    <child link="finger_link"/>
-    <origin rpy="0.0 -0.0 0.0" xyz="-0.035 0.0 0.0"/>
-    <axis xyz="1 0 0 "/>
-    <limit effort="1000.0" lower="-0.005" upper="0.035" velocity="0.1"/>
+    <parent link="base_link" />
+    <child link="finger_link" />
+    <origin rpy="0.0 -0.0 0.0" xyz="-0.035 0.0 0.0" />
+    <axis xyz="1 0 0 " />
+    <limit effort="1000.0" lower="-0.005" upper="0.035" velocity="0.1" />
   </joint>
   <!-- fixed joint to attach gripper to ur05 arm -->
@@ -61,5 +72,5 @@
     <parent link="ur5_tool0" />
     <child link="base_link" />
-    <origin rpy="${pi/2} 0.0 0.0" xyz="0.0 0.0 0.127"/>
+    <origin rpy="${pi/2} 0.0 0.0" xyz="0.0 0.0 0.127" />
   </joint>
   <ros2_control name="my_robot_arm" type="system">
@@ -67,54 +78,56 @@
       <plugin>gz_ros2_control/GazeboSimSystem</plugin>
     </hardware>
-    <xacro:property name="initial_positions_file" value="$(find my_robot_arm_moveit)/config/initial_positions.yaml" />
-    <xacro:property name="initial_positions" value="${xacro.load_yaml(initial_positions_file)['initial_positions']}"/>
+    <xacro:property name="initial_positions_file"
+      value="$(find my_robot_arm_moveit)/config/initial_positions.yaml" />
+    <xacro:property name="initial_positions"
+      value="${xacro.load_yaml(initial_positions_file)['initial_positions']}" />
     <joint name="ur5_shoulder_pan_joint">
-        <command_interface name="position"/>
-        <state_interface name="position">
-          <param name="initial_value">${initial_positions['ur5_shoulder_pan_joint']}</param>
-        </state_interface>
-        <state_interface name="velocity"/>
+      <command_interface name="position" />
+      <state_interface name="position">
+        <param name="initial_value">${initial_positions['ur5_shoulder_pan_joint']}</param>
+      </state_interface>
+      <state_interface name="velocity" />
     </joint>
     <joint name="ur5_shoulder_lift_joint">
-        <command_interface name="position"/>
-        <state_interface name="position">
-          <param name="initial_value">${initial_positions['ur5_shoulder_lift_joint']}</param>
-        </state_interface>
-        <state_interface name="velocity"/>
+      <command_interface name="position" />
+      <state_interface name="position">
+        <param name="initial_value">${initial_positions['ur5_shoulder_lift_joint']}</param>
+      </state_interface>
+      <state_interface name="velocity" />
     </joint>
     <joint name="ur5_elbow_joint">
-        <command_interface name="position"/>
-        <state_interface name="position">
-          <param name="initial_value">${initial_positions['ur5_elbow_joint']}</param>
-        </state_interface>
-        <state_interface name="velocity"/>
+      <command_interface name="position" />
+      <state_interface name="position">
+        <param name="initial_value">${initial_positions['ur5_elbow_joint']}</param>
+      </state_interface>
+      <state_interface name="velocity" />
     </joint>
     <joint name="ur5_wrist_1_joint">
-        <command_interface name="position"/>
-        <state_interface name="position">
-          <param name="initial_value">${initial_positions['ur5_wrist_1_joint']}</param>
-        </state_interface>
-        <state_interface name="velocity"/>
+      <command_interface name="position" />
+      <state_interface name="position">
+        <param name="initial_value">${initial_positions['ur5_wrist_1_joint']}</param>
+      </state_interface>
+      <state_interface name="velocity" />
     </joint>
     <joint name="ur5_wrist_2_joint">
-        <command_interface name="position"/>
-        <state_interface name="position">
-          <param name="initial_value">${initial_positions['ur5_wrist_2_joint']}</param>
-        </state_interface>
-        <state_interface name="velocity"/>
+      <command_interface name="position" />
+      <state_interface name="position">
+        <param name="initial_value">${initial_positions['ur5_wrist_2_joint']}</param>
+      </state_interface>
+      <state_interface name="velocity" />
     </joint>
     <joint name="ur5_wrist_3_joint">
-        <command_interface name="position"/>
-        <state_interface name="position">
-          <param name="initial_value">${initial_positions['ur5_wrist_3_joint']}</param>
-        </state_interface>
-        <state_interface name="velocity"/>
+      <command_interface name="position" />
+      <state_interface name="position">
+        <param name="initial_value">${initial_positions['ur5_wrist_3_joint']}</param>
+      </state_interface>
+      <state_interface name="velocity" />
     </joint>
     <joint name="finger_joint">
-        <command_interface name="position"/>
-        <state_interface name="position">
-          <param name="initial_value">${initial_positions['finger_joint']}</param>
-        </state_interface>
-        <state_interface name="velocity"/>
+      <command_interface name="position" />
+      <state_interface name="position">
+        <param name="initial_value">${initial_positions['finger_joint']}</param>
+      </state_interface>
+      <state_interface name="velocity" />
     </joint>
   </ros2_control>

Commit message: Day 17 - fix issue with realsense camera
In `src/my_robot_arm`package:

- in `CMakeLists.txt` and  `package.xml` - add dependency to
  `realsense2_description` package
- in`urdf/my_robot_arm.urdf.xacro` - add sensors plugin and
  relocate realsense camera to
    xyz=0 -1.6 0.6
    rpy=0 3*pi/4 -pi/2

File: src/my_robot_arm/urdf/my_robot_arm.urdf.xacro (robot description, xacro)
@@ -4,5 +4,5 @@
   <xacro:include filename="$(find sensors)/realsense_d435/realsense.urdf.xacro" />
   <xacro:realsense world_link_name="world">
-    <origin xyz="0 1.0 1.2" rpy="0 ${pi/4} -${pi/2}" />
+    <origin xyz="0 -1.6 0.6" rpy="0 ${3*pi/4} -${pi/2}" />
   </xacro:realsense>
   <!-- Include a UR05 -->
@@ -136,4 +136,7 @@
       <parameters>$(find my_robot_arm)/config/ros2_control.yaml</parameters>
     </plugin>
+    <plugin filename="gz-sim-sensors-system" name="gz::sim::systems::Sensors">
+      <render_engine>ogre2</render_engine>
+    </plugin>
   </gazebo>
 </robot>

Commit message: Day 18 (part 1) - configure collision avoidance  - in `src/my_robot_arm_moveit`:    - new config file `config/sensors_3d.yaml`- created by the Wizard
 - in `src/my_robot_arm`:
   - in `urdf/my_robot_arm.urdf.xacro` - move Realsense camera further
   away otherwise occupancy map does not work (seems to be a threshold
   for points closer than ~3m)

File: src/my_robot_arm/urdf/my_robot_arm.urdf.xacro (robot description, xacro)
@@ -4,5 +4,5 @@
   <xacro:include filename="$(find sensors)/realsense_d435/realsense.urdf.xacro" />
   <xacro:realsense world_link_name="world">
-    <origin xyz="0 -1.6 0.6" rpy="0 ${3*pi/4} -${pi/2}" />
+    <origin xyz="0 -3.0 1.8" rpy="0 ${3*pi/4} -${pi/2}" />
   </xacro:realsense>
   <!-- Include a UR05 -->
